Commit message: temporal

File: robots/TurtleBot2/turtlebot2_description/robots/kobuki_myrobot_d435_zed.urdf.xacro (robot description, xacro)
@@ -10,9 +10,12 @@
   <xacro:include filename="$(find turtlebot2_description)/urdf/stacks/myrobot.urdf.xacro"/>
   <xacro:include filename="$(find turtlebot2_description)/urdf/sensors/d435.urdf.xacro"/>
-  <!-- <xacro:include filename="$(find turtlebot_description)/urdf/sensors/kinect.urdf.xacro"/> -->
+  <xacro:include filename="$(find turtlebot2_description)/urdf/sensors/zed.urdf.xacro"/>
   <kobuki/>
-  <stack_myrobot parent="base_link"/>
-  <sensor_d435 parent="plate_top1_front_link"/>
-  <sensor_zed parent="plate_top2_front_link"/>
-  <!-- <sensor_kinect parent="base_link"/> -->
+  <xacro:stack_myrobot parent="base_link"/>
+  <xacro:sensor_d435 parent="plate_top1_front_link">
+    <origin xyz="0 0 0" rpy="0 0 0"/>
+  </xacro:sensor_d435>
+  <xacro:sensor_zed parent="plate_top2_front_link" camera_name="zed" camera_model="zed">
+    <origin xyz="0 0 0" rpy="0 0 0"/>
+  </xacro:sensor_zed>
 </robot>

File: robots/TurtleBot2/turtlebot2_description/urdf/stacks/myrobot.urdf.xacro (robot description, xacro)
@@ -7,6 +7,7 @@
   <!-- Xacro properties -->
   <xacro:property name="M_SCALE" value="0.001"/>
-  <xacro:property name="pole1_length" value="0.4" />
-  <xacro:property name="pole2_length" value="0.2032" />
+  <xacro:property name="default_top_pole_length" value="0.2032" />
+  <xacro:property name="pole1_length" value="0.2032" />
+  <xacro:property name="pole2_length" value="0.4" />
   <xacro:property name="plate_thickness" value="0.006" />
   <!-- Xacro macros -->
@@ -89,9 +90,9 @@
       </collision>
       <inertial>
-        <mass value="0.012"/>
-        <origin xyz="0 0 0"/>
-        <inertia ixx="0.000003805" ixy="0.0" ixz="0.0"
-                 iyy="0.000003805" iyz="0.0"
-                 izz="0.000000216"/>
+        <mass value="0.060"/>
+        <origin xyz="0 0 0"/>
+        <inertia ixx="0.000206991" ixy="0.0" ixz="0.0"
+                 iyy="0.000206991" iyz="0.0"
+                 izz="0.000001080"/>
       </inertial>
     </link>
@@ -107,34 +108,7 @@
         <origin xyz=" 0 0 0" rpy="0 0 0"/>
         <geometry>
-          <mesh filename="package://turtlebot_description/meshes/stacks/hexagons/pole_top.dae"/>
-        </geometry>
-      </visual>
-      <collision>
-        <origin xyz="0 0 0" rpy="0 0 0"/>
-        <geometry>
           <cylinder length="${pole2_length}" radius="0.006"/>
         </geometry>
-      </collision>
-      <inertial>
-        <mass value="0.060"/>
-        <origin xyz="0 0 0"/>
-        <inertia ixx="0.000206991" ixy="0.0" ixz="0.0"
-                 iyy="0.000206991" iyz="0.0"
-                 izz="0.000001080"/>
-      </inertial>
-    </link>
-  </xacro:macro>
-  <xacro:macro name="stack_top2_pole" params="parent number x_loc y_loc z_loc">
-    <joint name="pole_top_${number}_joint" type="fixed">
-      <origin xyz="${x_loc} ${y_loc} ${z_loc}" rpy="0 0 0"/>
-      <parent link="${parent}"/>
-      <child link="pole_top_${number}_link"/>
-    </joint>
-    <link name="pole_top_${number}_link">
-      <visual>
-        <origin xyz=" 0 0 0" rpy="0 0 0"/>
-        <geometry>
-          <mesh filename="package://turtlebot_description/meshes/stacks/hexagons/pole_top.dae"/>
-        </geometry>
+        <material name="gray"/>
       </visual>
       <collision>
@@ -221,10 +195,10 @@
       </inertial>
     </link>
-    <stack_top1_pole parent="${parent}" number="0" x_loc= "0.0381" y_loc= "0.1505" z_loc="${0.2920 - pole2_length/2.0 + pole1_length/2.0}"/>
-    <stack_top1_pole parent="${parent}" number="1" x_loc= "0.0381" y_loc="-0.1505" z_loc="${0.2920 - pole2_length/2.0 + pole1_length/2.0}"/>
-    <stack_top1_pole parent="${parent}" number="2" x_loc="-0.0381" y_loc= "0.1505" z_loc="${0.2920 - pole2_length/2.0 + pole1_length/2.0}"/>
-    <stack_top1_pole parent="${parent}" number="3" x_loc="-0.0381" y_loc="-0.1505" z_loc="${0.2920 - pole2_length/2.0 + pole1_length/2.0}"/>
+    <stack_top1_pole parent="${parent}" number="0" x_loc= "0.0381" y_loc= "0.1505" z_loc="${0.2920 - default_top_pole_length/2.0 + pole1_length/2.0}"/>
+    <stack_top1_pole parent="${parent}" number="1" x_loc= "0.0381" y_loc="-0.1505" z_loc="${0.2920 - default_top_pole_length/2.0 + pole1_length/2.0}"/>
+    <stack_top1_pole parent="${parent}" number="2" x_loc="-0.0381" y_loc= "0.1505" z_loc="${0.2920 - default_top_pole_length/2.0 + pole1_length/2.0}"/>
+    <stack_top1_pole parent="${parent}" number="3" x_loc="-0.0381" y_loc="-0.1505" z_loc="${0.2920 - default_top_pole_length/2.0 + pole1_length/2.0}"/>
     <joint name="plate_top1_joint" type="fixed">
-      <origin xyz="-0.01364 0.0  ${0.2920 - pole2_length/2.0 + pole1_length + plate_thickness/2.0}" rpy="0 0 0"/>
+      <origin xyz="-0.01364 0.0  ${0.2920 - default_top_pole_length/2.0 + pole1_length + plate_thickness/2.0}" rpy="0 0 0"/>
       <parent link="${parent}"/>
       <child link="plate_top1_link"/>
@@ -251,10 +225,10 @@
       </inertial>
     </link>
-    <stack_top2_pole parent="${parent}" number="0" x_loc= "0.0381" y_loc= "0.1505" z_loc="${0.2920 + pole1_length + plate_thickness}"/>
-    <stack_top2_pole parent="${parent}" number="1" x_loc= "0.0381" y_loc="-0.1505" z_loc="${0.2920 + pole1_length + plate_thickness}"/>
-    <stack_top2_pole parent="${parent}" number="2" x_loc="-0.0381" y_loc= "0.1505" z_loc="${0.2920 + pole1_length + plate_thickness}"/>
-    <stack_top2_pole parent="${parent}" number="3" x_loc="-0.0381" y_loc="-0.1505" z_loc="${0.2920 + pole1_length + plate_thickness}"/>
+    <stack_top2_pole parent="${parent}" number="0" x_loc= "0.0381" y_loc= "0.1505" z_loc="${0.2920 - default_top_pole_length/2.0 + pole1_length + pole2_length/2.0 + plate_thickness}"/>
+    <stack_top2_pole parent="${parent}" number="1" x_loc= "0.0381" y_loc="-0.1505" z_loc="${0.2920 - default_top_pole_length/2.0 + pole1_length + pole2_length/2.0 + plate_thickness}"/>
+    <stack_top2_pole parent="${parent}" number="2" x_loc="-0.0381" y_loc= "0.1505" z_loc="${0.2920 - default_top_pole_length/2.0 + pole1_length + pole2_length/2.0 + plate_thickness}"/>
+    <stack_top2_pole parent="${parent}" number="3" x_loc="-0.0381" y_loc="-0.1505" z_loc="${0.2920 - default_top_pole_length/2.0 + pole1_length + pole2_length/2.0 + plate_thickness}"/>
     <joint name="plate_top2_joint" type="fixed">
-      <origin xyz="-0.01364 0.0  ${0.2920 + pole1_length + plate_thickness + pole2_length/2.0 + plate_thickness/2.0}" rpy="0 0 0"/>
+      <origin xyz="-0.01364 0.0  ${0.2920 - default_top_pole_length/2.0 + pole1_length + plate_thickness + pole2_length + plate_thickness/2.0}" rpy="0 0 0"/>
       <parent link="${parent}"/>
       <child link="plate_top2_link"/>
@@ -297,6 +271,6 @@
     <!-- joint for D435 camera -->
     <joint name="plate_top1_front_joint" type="fixed">
-      <origin xyz="${0.003 + 0.09525} 0.0  ${0.2920 - pole2_length/2.0 + pole1_length + plate_thickness/2.0}" rpy="0 0 0"/>
-      <parent link="${parent}"/>
+      <origin xyz="${0.003 + 0.09525} 0.0  ${plate_thickness/2.0}" rpy="0 0 0"/>
+      <parent link="plate_top1_link"/>
       <child link="plate_top1_front_link"/>
     </joint>
@@ -306,6 +280,6 @@
     <!-- joint for ZED camera -->
     <joint name="plate_top2_front_joint" type="fixed">
-      <origin xyz="${0.003 + 0.09525} 0.0  ${0.2920 + pole1_length + plate_thickness + pole2_length/2.0 + plate_thickness/2.0}" rpy="0 0 0"/>
-      <parent link="${parent}"/>
+      <origin xyz="${0.003 + 0.09525} 0.0  ${plate_thickness/2.0}" rpy="0 0 0"/>
+      <parent link="plate_top2_link"/>
       <child link="plate_top2_front_link"/>
     </joint>
