Commit message: [add] add vlp-16 to myrobot

File: robots/TurtleBot2/turtlebot2_description/robots/kobuki_myrobot_d455_d455_vlp16.urdf.xacro (robot description, xacro)
@@ -10,4 +10,5 @@
   <xacro:include filename="$(find turtlebot2_description)/urdf/stacks/myrobot.urdf.xacro"/>
   <xacro:include filename="$(find turtlebot2_description)/urdf/sensors/d455.urdf.xacro"/>
+  <xacro:include filename="$(find velodyne_description)/urdf/VLP-16.urdf.xacro"/>
   <kobuki/>
   <xacro:stack_myrobot parent="base_link"/>
@@ -18,3 +19,6 @@
     <origin xyz="0 0 0" rpy="0 0 0"/>
   </xacro:sensor_d455>
+  <xacro:VLP-16 parent="plate_top2_center_link" name="velodyne" topic="/velodyne_points" noise="0.008" gpu="true">
+    <origin xyz="0 0 0" rpy="0 0 0"/>
+  </xacro:VLP-16>
 </robot>

File: robots/TurtleBot2/turtlebot2_description/urdf/stacks/myrobot.urdf.xacro (robot description, xacro)
@@ -262,12 +262,13 @@
     <link name="plate_top1_center_link">
     </link> -->
-    <!-- <joint name="plate_top2_center_joint" type="fixed">
-      <origin xyz="0.003 0.0  ${0.2920 + pole1_length + plate_thickness + pole2_length/2.0 + plate_thickness/2.0}" rpy="0 0 0"/>
-      <parent link="${parent}"/>
+    <!-- joint for VLP-16  on the plate_top2 -->
+    <joint name="plate_top2_center_joint" type="fixed">
+      <origin xyz="0.003 0.0  ${plate_thickness/2.0}" rpy="0 0 0"/>
+      <parent link="plate_top2_link"/>
       <child link="plate_top2_center_link"/>
     </joint>
     <link name="plate_top2_center_link">
-    </link> -->
-    <!-- joint for D435 camera -->
+    </link>
+    <!-- joint for D455_top1 camera on the plate_top1 -->
     <joint name="plate_top1_front_joint" type="fixed">
       <origin xyz="${0.003 + 0.09525} 0.0  ${plate_thickness/2.0}" rpy="0 0 0"/>
@@ -276,7 +277,6 @@
     </joint>
     <link name="plate_top1_front_link">
-      <!-- include d435 xacro -->
-    </link>
-    <!-- joint for ZED camera -->
+    </link>
+    <!-- joint for D455_top2 camera on the plate_top2 -->
     <joint name="plate_top2_front_joint" type="fixed">
       <origin xyz="${0.003 + 0.09525} 0.0  ${plate_thickness/2.0}" rpy="0 0 0"/>
@@ -285,5 +285,4 @@
     </joint>
     <link name="plate_top2_front_link">
-      <!-- include zed xacro -->
     </link>
   </xacro:macro>
